Commit message: added all urdf files and launches

File: sim_robot/description/robot.urdf.xacro (robot description, xacro)
@@ -1,6 +1,15 @@
 <?xml version="1.0"?>
 <robot xmlns:xacro="http://www.ros.org/wiki/xacro"  name="robot">
-    <xacro:arg name="use_ros2_control" default="true"/>
+    <xacro:arg name="use_ros2_control" default="false"/>
     <xacro:arg name="sim_mode" default="true"/>
     <xacro:include filename="robot_core.xacro"/>
+    <xacro:include filename="lidar.xacro"/>
+    <!-- <xacro:include filename="gazebo_control.xacro" /> -->
+    <xacro:include filename="ros2_control.xacro" />
+     <!-- <xacro:if value="$(arg use_ros2_control)">
+        <xacro:include filename="ros2_control.xacro" />
+    </xacro:if>
+    <xacro:unless value="$(arg use_ros2_control)">
+        <xacro:include filename="gazebo_control.xacro" />
+    </xacro:unless>  -->
 </robot>

File: sim_robot/description/robot_core.xacro (robot description, xacro)
@@ -31,4 +31,5 @@
     <xacro:property name="wheel_offset_y" value="0.166"/>
     <xacro:property name="wheel_offset_z" value="0.01"/>
+    <xacro:property name="max_steer" value="0.6458"/>
 	<!-- Base link -->
   <link name="base_link">
@@ -59,7 +60,4 @@
     </link>
     <gazebo reference="chasis">
-        <material> Gazebo/White</material>
-    </gazebo>
-    <!-- <gazebo reference="chassis">
         <kp>1000000.0</kp>
         <kd>0.1</kd>
@@ -71,5 +69,5 @@
         <mu2 value="0.1"/>
         <fdir1 value="0 0 0"/>
-    </gazebo>  -->
+    </gazebo>
     <!--FRONT RIGHT WHEEL ROTATE-->
     <joint name="front_right_wheel_rotate_joint" type="revolute">
@@ -77,6 +75,6 @@
         <child link="front_right_wheel_rotate"/>
         <origin xyz="${front_rear_sep + (chasis_x - front_rear_sep)/2} -${wheel_sep/2 + wheel_thickness} 0" rpy="0 0 0" />
-        <axis xyz="0 0 -1"/>
-        <limit effort="100" velocity="1" lower="-1" upper="1"/>
+        <axis xyz="0 0 1"/>
+        <limit effort="100" velocity="1" lower="-${max_steer}" upper="${max_steer}"/>
     </joint>
     <link name="front_right_wheel_rotate">
@@ -99,14 +97,11 @@
 	</link>
     <gazebo reference="front_right_wheel_rotate">
-        <material>Gazebo/Blue</material>
-    </gazebo>
-    <!-- <gazebo reference="right_wheel_rotate">
-    <mu1 value="2.0"/>
-    <mu2 value="2.0"/>
-    <kp  value="10000000.0" />
-    <kd  value="1.0" />
-    <fdir1 value="0 1 0"/>
-    <material>Gazebo/White</material>
-    </gazebo> -->
+        <mu1 value="2.0"/>
+        <mu2 value="2.0"/>
+        <kp  value="10000000.0" />
+        <kd  value="1.0" />
+        <fdir1 value="0 1 0"/>
+        <material>Gazebo/Blue</material>
+      </gazebo>
     <!--FRONT RIGHT WHEEL MOVE-->
     <joint name="front_right_wheel_move_joint" type="continuous">
@@ -133,14 +128,11 @@
 	</link>
     <gazebo reference="front_right_wheel_move">
-        <material>Gazebo/Blue</material>
-    </gazebo>
-    <!-- <gazebo reference="right_wheel">
-    <mu1 value="2.0"/>
-    <mu2 value="2.0"/>
-    <kp  value="10000000.0" />
-    <kd  value="1.0" />
-    <fdir1 value="0 1 0"/>
-    <material>Gazebo/Blue</material>
-    </gazebo> -->
+        <mu1 value="2.0"/>
+        <mu2 value="2.0"/>
+        <kp  value="10000000.0" />
+        <kd  value="1.0" />
+        <fdir1 value="0 1 0"/>
+        <material>Gazebo/Blue</material>
+    </gazebo>
     <!--FRONT LEFT WHEEL ROTATE-->
     <joint name="front_left_wheel_rotate_joint" type="revolute">
@@ -149,5 +141,5 @@
         <origin xyz="${front_rear_sep + (chasis_x - front_rear_sep)/2} ${wheel_sep/2 + wheel_thickness} 0" rpy="0 0 0" />
         <axis xyz="0 0 1"/>
-        <limit effort="100" velocity="1" lower="-1" upper="1"/>
+        <limit effort="100" velocity="1" lower="-${max_steer}" upper="${max_steer}"/>
     </joint>
     <link name="front_left_wheel_rotate">
@@ -170,14 +162,11 @@
 	</link>
     <gazebo reference="front_left_wheel_rotate">
-        <material>Gazebo/Blue</material>
-    </gazebo>
-    <!-- <gazebo reference="left_wheel_rotate">
-    <mu1 value="2.0"/>
-    <mu2 value="2.0"/>
-    <kp  value="10000000.0" />
-    <kd  value="1.0" />
-    <fdir1 value="0 1 0"/>
-    <material>Gazebo/White</material>
-    </gazebo> -->
+        <mu1 value="2.0"/>
+        <mu2 value="2.0"/>
+        <kp  value="10000000.0" />
+        <kd  value="1.0" />
+        <fdir1 value="0 1 0"/>
+        <material>Gazebo/Blue</material>
+      </gazebo>
     <!--LEFT RIGHT WHEEL MOVE-->
     <joint name="front_left_wheel_move_joint" type="continuous">
@@ -204,15 +193,11 @@
 	</link>
     <gazebo reference="front_left_wheel_move">
-        <material>Gazebo/Blue</material>
-    </gazebo>
-    <!-- <gazebo reference="left_wheel">
-    <mu1 value="2.0"/>
-    <mu2 value="2.0"/>
-    <kp  value="10000000.0" />
-    <kd  value="1.0" />
-    <fdir1 value="0 1 0"/>
-    <material>Gazebo/Blue</material>
-    </gazebo> -->
-    <!-- HASTA AQUI -->
+        <mu1 value="2.0"/>
+        <mu2 value="2.0"/>
+        <kp  value="10000000.0" />
+        <kd  value="1.0" />
+        <fdir1 value="0 1 0"/>
+        <material>Gazebo/White</material>
+      </gazebo>
     <!--BACK RIGHT WHEEL-->
     <joint name="back_right_wheel_joint" type="continuous">
@@ -221,5 +206,4 @@
         <origin xyz="${(chasis_x - front_rear_sep)/2} -${wheel_sep/2 + wheel_thickness} 0" rpy="${pi/2} 0 0" />
         <axis xyz="0 0 -1"/>
-        <limit effort="100" velocity="1" lower="-1" upper="1"/>
     </joint>
     <link name="back_right_wheel">
@@ -240,14 +224,11 @@
 	</link>
     <gazebo reference="back_right_wheel">
-        <material>Gazebo/Blue</material>
-    </gazebo>
-    <!-- <gazebo reference="right_wheel_rotate">
-    <mu1 value="2.0"/>
-    <mu2 value="2.0"/>
-    <kp  value="10000000.0" />
-    <kd  value="1.0" />
-    <fdir1 value="0 1 0"/>
-    <material>Gazebo/White</material>
-    </gazebo> -->
+        <mu1 value="2.0"/>
+        <mu2 value="2.0"/>
+        <kp  value="10000000.0" />
+        <kd  value="1.0" />
+        <fdir1 value="0 1 0"/>
+        <material>Gazebo/Blue</material>
+      </gazebo>
     <!--BACK LEFT WHEEL-->
     <joint name="back_left_wheel_joint" type="continuous">
@@ -256,5 +237,4 @@
         <origin xyz="${(chasis_x - front_rear_sep)/2} ${wheel_sep/2 + wheel_thickness} 0" rpy="-${pi/2} 0 0" />
         <axis xyz="0 0 1"/>
-        <limit effort="100" velocity="1" lower="-1" upper="1"/>
     </joint>
     <link name="back_left_wheel">
@@ -277,11 +257,11 @@
         <material>Gazebo/Blue</material>
     </gazebo>
-    <!-- <gazebo reference="left_wheel_rotate">
-    <mu1 value="2.0"/>
-    <mu2 value="2.0"/>
-    <kp  value="10000000.0" />
-    <kd  value="1.0" />
-    <fdir1 value="0 1 0"/>
-    <material>Gazebo/White</material>
-    </gazebo> -->
+    <gazebo reference="left_wheel_rear">
+        <mu1 value="2.0"/>
+        <mu2 value="2.0"/>
+        <kp  value="10000000.0" />
+        <kd  value="1.0" />
+        <fdir1 value="0 1 0"/>
+        <material>Gazebo/Blue</material>
+    </gazebo>
 	</robot>
