Commit message: added ackerman params for nav2

File: sim_robot/description/gazebo_control.xacro (robot description, xacro)
@@ -11,6 +11,6 @@
                 <right_steering_joint>front_right_wheel_rotate_joint</right_steering_joint>
                 <steering_wheel_joint>front_right_wheel_rotate_joint</steering_wheel_joint>
-                <wheel_radius>0.05</wheel_radius>
-                <wheel_separation>0.36</wheel_separation>
+                <wheel_radius>0.155</wheel_radius>
+                <wheel_separation>0.6</wheel_separation>
                 <!-- Max absolute steer angle for tyre in radians-->
                 <!-- Any cmd_vel angular z greater than this would be capped -->

File: sim_robot/description/robot.urdf.xacro (robot description, xacro)
@@ -6,4 +6,5 @@
     <xacro:include filename="lidar.xacro"/>
     <xacro:include filename="gps.xacro"/>
+    <xacro:include filename="imu.xacro"/>
     <!-- <xacro:include filename="gazebo_control.xacro" /> -->
     <xacro:include filename="ros2_control.xacro" />
@@ -12,5 +13,5 @@
     </xacro:if>
     <xacro:unless value="$(arg use_ros2_control)">
-        <xacro:include filename="gazebo_control.xacro" />
+         />
     </xacro:unless>  -->
 </robot>

File: sim_robot/description/robot_core.xacro (robot description, xacro)
@@ -19,20 +19,23 @@
     </material>
     <!-- PROPERTIES FOR SIZES -->
-    <xacro:property name="chasis_x" value="0.6"/>
-    <xacro:property name="chasis_y" value="0.3"/>
-    <xacro:property name="chasis_z" value="0.2"/>
-    <xacro:property name="chasis_mass" value="1.0"/>
-    <xacro:property name="wheel_radius" value="0.05"/>
-    <xacro:property name="wheel_thickness" value="0.03"/>
-    <xacro:property name="wheel_sep" value="0.3"/>
-    <xacro:property name="front_rear_sep" value="0.5"/>
-    <xacro:property name="wheel_mass" value="0.05"/>
-    <xacro:property name="wheel_offset_x" value="0.226"/>
-    <xacro:property name="wheel_offset_y" value="0.166"/>
-    <xacro:property name="wheel_offset_z" value="0.01"/>
+    <xacro:property name="chasis_x" value="0.94"/>
+    <xacro:property name="chasis_y" value="0.39"/>
+    <xacro:property name="chasis_z" value="0.28"/>
+    <xacro:property name="chasis_mass" value="50.0"/>
+    <xacro:property name="wheel_radius" value="0.155"/>
+    <xacro:property name="wheel_thickness" value="0.14"/>
+    <xacro:property name="wheel_sep" value="0.6"/>
+    <xacro:property name="front_rear_sep" value="0.65"/>
+    <xacro:property name="wheel_mass" value="0.5"/>
     <xacro:property name="max_steer" value="0.6458"/>
 	<!-- Base link -->
-  <link name="base_link">
-  </link>
+    <link name="base_footprint"/>
+    <joint name="base_joint" type="fixed">
+        <parent link="base_footprint"/>
+        <child link="base_link" />
+        <origin xyz="0 0 0" rpy="0 0 0"/>
+      </joint>
+    <link name="base_link">
+    </link>
 	<!-- Chasis-->
 	<joint name="chasis_joint" type="fixed">

File: sim_robot/description/ros2_control.xacro (robot description, xacro)
@@ -58,4 +58,5 @@
                 <remapping>ack_cont/odometry:=odom</remapping>
                 <remapping>ack_cont/tf_odometry:=tf</remapping>
+                <remapping>ack_cont/reference_unstamped:=cmd_vel</remapping>
             </ros>
             <parameters>$(find sim_robot)/config/my_controllers.yaml</parameters>
