Commit message: borrado el pkg de mqtt

File: hunter_sim_pkg/description/hunter2.xacro (robot description, xacro)
@@ -1,32 +1,14 @@
 <?xml version="1.0" encoding="utf-8"?>
-<!-- This URDF was automatically created by SolidWorks to URDF Exporter! Originally created by Stephen Brawner (brawner@gmail.com)
-     Commit Version: 1.6.0-1-g15f4949  Build Version: 1.6.7594.29634
-     For more information, please see http://wiki.ros.org/sw_urdf_exporter -->
-<robot
-  name="hunter2_base" xmlns:xacro="http://www.ros.org/wiki/xacro">
-  <xacro:include filename="inertial_macros.xacro"/>
-  <material name="white">
-    <color rgba="1 1 1 1"/>
-</material>
-<material name="orange">
-    <color rgba="1 0.3 0.1 1"/>
-</material>
-<material name="blue">
-    <color rgba="0.2 0.2 1 1"/>
-</material>
-<material name="black">
-    <color rgba="0 0 0 1"/>
-</material>
-<material name="red">
-    <color rgba="1 0 0 1"/>
-</material>
-  <link
-    name="base_link">
-    <inertial>
-      <origin
-        xyz="0.0266989327622036 0.000409203500587652 -0.135901124750884"
-        rpy="0 0 0" />
-      <mass
-        value="21.02945169536679" />
+<robot name="hunter">
+  <link name="base_footprint">
+  </link>
+  <joint name="base_link_footprint_joint" type="fixed">
+    <parent link="base_footprint"/>
+    <child link="base_link"/>
+  </joint>
+  <link name="base_link">
+    <inertial>
+      <origin xyz="0 0 0" rpy="0 0 0" />
+      <mass value="21.02945169536679" />
       <inertia
         ixx="0.0332370959804736"
@@ -43,5 +25,5 @@
       <geometry>
         <mesh
-          filename="package://hunter_sim_pkg/mesh/meshes/base_link.STL" />
+          filename="package://tfg_pkg/meshes/base_link.STL" />
       </geometry>
       <material
@@ -57,19 +39,8 @@
       <geometry>
         <mesh
-          filename="package://hunter_sim_pkg/mesh/meshes/base_link.STL" />
-      </geometry>
-    </collision>
-  </link>
-  <gazebo reference="base_link">
-    <kp>1000000.0</kp>
-    <kd>0.1</kd>
-    <dampingFactor>0</dampingFactor>
-    <material>Gazebo/White</material>
-    <selfCollide>true</selfCollide>
-    <turnGravityOff>false</turnGravityOff>
-    <mu1 value="0.5"/>
-    <mu2 value="0.5"/>
-    <fdir1 value="0 0 0"/>
-  </gazebo>
+          filename="package://tfg_pkg/meshes/base_link.STL" />
+      </geometry>
+    </collision>
+  </link>
   <link
     name="front_steer_left_link">
@@ -78,6 +49,5 @@
         xyz="-0.012614 1.8116E-05 0.0023132"
         rpy="0 0 0" />
-      <mass
-        value="7.8526" />
+      <mass value="7.8526" />
       <inertia
         ixx="0.063827"
@@ -128,12 +98,4 @@
       velocity="0" />
   </joint>
-  <gazebo reference="front_steer_left_link">
-        <mu1 value="0.5"/>
-        <mu2 value="0.5"/>
-        <kp  value="10000000.0" />
-        <kd  value="1.0" />
-        <fdir1 value="0 1 0"/>
-        <material>Gazebo/Blue</material>
-      </gazebo>
   <link
     name="front_left_wheel_link">
@@ -158,19 +120,19 @@
       <geometry>
         <mesh
-          filename="package://hunter_sim_pkg/mesh/meshes/front_left_wheel_link.STL" />
-      </geometry>
-      <material
-        name="">
-        <color
-          rgba="0.79216 0.81961 0.93333 1" />
-      </material>
-    </visual>
-    <collision>
-      <origin
-        xyz="0 0 0"
-        rpy="0 0 0" />
-      <geometry>
-        <mesh
-          filename="package://hunter_sim_pkg/mesh/meshes/front_left_wheel_link.STL" />
+          filename="package://tfg_pkg/meshes/front_left_wheel_link.STL" />
+      </geometry>
+      <material
+        name="">
+        <color
+          rgba="0.79216 0.81961 0.93333 1" />
+      </material>
+    </visual>
+    <collision>
+      <origin
+        xyz="0 0 0"
+        rpy="0 0 0" />
+      <geometry>
+        <mesh
+          filename="package://tfg_pkg/meshes/front_left_wheel_link.STL" />
       </geometry>
     </collision>
@@ -190,12 +152,4 @@
       <dynamics damping="0.0" friction="15"/>
   </joint>
-  <gazebo reference="front_left_wheel_link">
-    <mu1 value="0.5"/>
-    <mu2 value="0.5"/>
-    <kp  value="10000000.0" />
-    <kd  value="1.0" />
-    <fdir1 value="0 1 0"/>
-    <material>Gazebo/Blue</material>
-  </gazebo>
   <link
     name="front_steer_right_link">
@@ -254,12 +208,4 @@
       velocity="0" />
   </joint>
-  <gazebo reference="front_steer_right_link">
-    <mu1 value="0.5"/>
-    <mu2 value="0.5"/>
-    <kp  value="10000000.0" />
-    <kd  value="1.0" />
-    <fdir1 value="0 1 0"/>
-    <material>Gazebo/Blue</material>
-  </gazebo>
   <link
     name="front_right_wheel_link">
@@ -284,19 +230,19 @@
       <geometry>
         <mesh
-          filename="package://hunter_sim_pkg/mesh/meshes/front_left_wheel_link.STL" />
-      </geometry>
-      <material
-        name="">
-        <color
-          rgba="0.79216 0.81961 0.93333 1" />
-      </material>
-    </visual>
-    <collision>
-      <origin
-        xyz="0 0 0"
-        rpy="0 0 0" />
-      <geometry>
-        <mesh
-          filename="package://hunter_sim_pkg/mesh/meshes/front_right_wheel_link.STL" />
+          filename="package://tfg_pkg/meshes/front_right_wheel_link.STL" />
+      </geometry>
+      <material
+        name="">
+        <color
+          rgba="0.79216 0.81961 0.93333 1" />
+      </material>
+    </visual>
+    <collision>
+      <origin
+        xyz="0 0 0"
+        rpy="0 0 0" />
+      <geometry>
+        <mesh
+          filename="package://tfg_pkg/meshes/front_right_wheel_link.STL" />
       </geometry>
     </collision>
@@ -316,12 +262,4 @@
       <dynamics damping="0.0" friction="15"/>
   </joint>
-  <gazebo reference="front_right_wheel_link">
-    <mu1 value="0.5"/>
-    <mu2 value="0.5"/>
-    <kp  value="10000000.0" />
-    <kd  value="1.0" />
-    <fdir1 value="0 1 0"/>
-    <material>Gazebo/Blue</material>
-  </gazebo>
   <link
     name="left_rear_link">
@@ -346,19 +284,19 @@
       <geometry>
         <mesh
-          filename="package://hunter_sim_pkg/mesh/meshes/left_rear_link.STL" />
-      </geometry>
-      <material
-        name="">
-        <color
-          rgba="0.79216 0.81961 0.93333 1" />
-      </material>
-    </visual>
-    <collision>
-      <origin
-        xyz="0 0 0"
-        rpy="0 0 0" />
-      <geometry>
-        <mesh
-          filename="package://hunter_sim_pkg/mesh/meshes/left_rear_link.STL" />
+          filename="package://tfg_pkg/meshes/left_rear_link.STL" />
+      </geometry>
+      <material
+        name="">
+        <color
+          rgba="0.79216 0.81961 0.93333 1" />
+      </material>
+    </visual>
+    <collision>
+      <origin
+        xyz="0 0 0"
+        rpy="0 0 0" />
+      <geometry>
+        <mesh
+          filename="package://tfg_pkg/meshes/left_rear_link.STL" />
       </geometry>
     </collision>
@@ -378,12 +316,4 @@
      <dynamics damping="0.0" friction="15"/>
   </joint>
-  <gazebo reference="left_rear_link">
-    <mu1 value="0.5"/>
-    <mu2 value="0.5"/>
-    <kp  value="10000000.0" />
-    <kd  value="1.0" />
-    <fdir1 value="0 1 0"/>
-    <material>Gazebo/Blue</material>
-  </gazebo>
   <link
     name="right_rear_link">
@@ -408,19 +338,19 @@
       <geometry>
         <mesh
-          filename="package://hunter_sim_pkg/mesh/meshes/right_rear_link.STL" />
-      </geometry>
-      <material
-        name="">
-        <color
-          rgba="0.79216 0.81961 0.93333 1" />
-      </material>
-    </visual>
-    <collision>
-      <origin
-        xyz="0 0 0"
-        rpy="0 0 0" />
-      <geometry>
-        <mesh
-          filename="package://hunter_sim_pkg/mesh/meshes/right_rear_link.STL" />
+          filename="package://tfg_pkg/meshes/right_rear_link.STL" />
+      </geometry>
+      <material
+        name="">
+        <color
+          rgba="0.79216 0.81961 0.93333 1" />
+      </material>
+    </visual>
+    <collision>
+      <origin
+        xyz="0 0 0"
+        rpy="0 0 0" />
+      <geometry>
+        <mesh
+          filename="package://tfg_pkg/meshes/right_rear_link.STL" />
       </geometry>
     </collision>
@@ -440,386 +370,16 @@
      <dynamics damping="0.0" friction="15"/>
   </joint>
-  <gazebo reference="right_rear_link">
-    <mu1 value="0.5"/>
-    <mu2 value="0.5"/>
-    <kp  value="10000000.0" />
-    <kd  value="1.0" />
-    <fdir1 value="0 1 0"/>
-    <material>Gazebo/Blue</material>
-  </gazebo>
-  <link
-    name="front_steer_link">
-    <inertial>
-      <origin
-        xyz="0.049836 8.1046E-15 0.017912"
-        rpy="0 0 0" />
-      <mass
-        value="0.0049179" />
-      <inertia
-        ixx="1.6846E-07"
-        ixy="7.6396E-23"
-        ixz="-1.0974E-08"
-        iyy="7.549E-07"
-        iyz="-1.8957E-22"
-        izz="7.334E-07" />
-    </inertial>
-    <visual>
-      <origin
-        xyz="0 0 0"
-        rpy="0 0 0" />
-      <geometry>
-      <cylinder length="0.001" radius="0.005"/>
-      </geometry>
-      <material
-        name="">
-        <color
-          rgba="0.79216 0.81961 0.93333 1" />
-      </material>
-    </visual>
-    <collision>
-      <origin
-        xyz="0 0 0"
-        rpy="0 0 0" />
-      <geometry>
-      <cylinder length="0.001" radius="0.005"/>
-      </geometry>
-    </collision>
-  </link>
-  <joint
-    name="front_steer_joint"
-    type="revolute">
-    <origin
-      xyz="0.44792 -1.1431E-05 -0.121"
-      rpy="0 0 0" />
-    <parent
-      link="base_link" />
-    <child
-      link="front_steer_link" />
-    <axis
-      xyz="0 0 1" />
-    <limit
-      lower="-0.72"
-      upper="0.72"
-      effort="0"
-      velocity="0" />
-  </joint>
-  <gazebo reference="front_steer_link">
-    <mu1 value="0.5"/>
-    <mu2 value="0.5"/>
-    <kp  value="10000000.0" />
-    <kd  value="1.0" />
-    <fdir1 value="0 1 0"/>
-    <material>Gazebo/Blue</material>
-  </gazebo>
-  <link
-    name="rear_wheel_link">
-    <inertial>
-      <origin
-        xyz="-0.02 0.0031269 -0.12735"
-        rpy="0 0 0" />
-      <mass
-        value="0.0049179" />
-      <inertia
-        ixx="1.1821E-06"
-        ixy="9.6965E-13"
-        ixz="-3.1553E-12"
-        iyy="9.5276E-07"
-        iyz="1.2428E-08"
-        izz="1.0913E-06" />
-    </inertial>
-    <visual>
-      <origin
-        xyz="0 0 0"
-        rpy="0 0 0" />
-      <geometry>
-      <cylinder length="0.001" radius="0.005"/>
-      </geometry>
-      <material
-        name="">
-        <color
-          rgba="1 1 1 1" />
-      </material>
-    </visual>
-    <collision>
-      <origin
-        xyz="0 0 0"
-        rpy="0 0 0" />
-      <geometry>
-      <cylinder length="0.001" radius="0.005"/>
-      </geometry>
-    </collision>
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
File: hunter_sim_pkg/description/simple_urdf/robot_core.xacro (robot description, xacro)
@@ -38,5 +38,4 @@
         <parent link="base_link"/>
         <child link="chasis"/>
-        <origin xyz="-${chasis_x/2} 0 0"/>
     </joint>
     <link name="chasis">
@@ -54,7 +53,14 @@
         </geometry>
         </collision>
-        <xacro:inertial_box mass="${chasis_mass}" x="${chasis_x}" y="${chasis_y}" z="${chasis_z}">
-                <origin xyz="${chasis_x/2} 0 ${chasis_z/2}" rpy="0 0 0"/>
-        </xacro:inertial_box>
+        <inertial>
+            <mass value="21.02945169536679" />
+            <inertia
+              ixx="0.0332370959804736"
+              ixy="-1.013150489971E-06"
+              ixz="-0.00188859201421112"
+              iyy="0.111072002332437"
+              iyz="-5.13308150598312E-07"
+              izz="0.12660862809283" />
+          </inertial>
     </link>
     <gazebo reference="chasis">
@@ -75,5 +81,9 @@
         <origin xyz="${front_rear_sep + (chasis_x - front_rear_sep)/2} -${wheel_sep/2 + wheel_thickness} 0" rpy="0 0 0" />
         <axis xyz="0 0 1"/>
-        <limit effort="100" velocity="1" lower="-${max_steer}" upper="${max_steer}"/>
+        <limit
+      lower="-0.69"
+      upper="0.69"
+      effort="0"
+      velocity="0" />
     </joint>
     <link name="front_right_wheel_rotate">
@@ -88,10 +98,18 @@
             <origin xyz="0 0 0" rpy="${pi/2} 0 0" />
 		    <geometry>
-                <cylinder length="${wheel_thickness}" radius="${wheel_radius}"/>
-            </geometry>
-		</collision>
-		<xacro:inertial_cylinder mass="${wheel_mass}" length="${wheel_thickness}" radius="${wheel_radius}">
-            <origin xyz="0 0 0" rpy="${pi/2} 0 0"/>
-        </xacro:inertial_cylinder>
+                <sphere  radius="${wheel_radius}"/>
+            </geometry>
+		</collision>
+		<inertial>
+            <mass
+              value="7.696" />
+            <inertia
+              ixx="0.063704"
+              ixy="0"
+              ixz="0"
+              iyy="0.063704"
+              iyz="0"
+              izz="0.11068" />
+          </inertial>
 	</link>
     <gazebo reference="front_right_wheel_rotate">
@@ -109,4 +127,5 @@
         <origin xyz="0 0 0" rpy="${pi/2} 0 0" />
         <axis xyz="0 0 -1" rpy="0 0 0" />
+        <dynamics damping="0.0" friction="15"/>
     </joint>
 	<link name="front_right_wheel_move">
@@ -119,10 +138,18 @@
 		<collision>
 		    <geometry>
-                <cylinder length="${wheel_thickness}" radius="${wheel_radius}"/>
+                <sphere radius="${wheel_radius}"/>
 		    </geometry>
 		</collision>
-        <xacro:inertial_cylinder mass="${wheel_mass}" length="${wheel_thickness}" radius="${wheel_radius}">
-            <origin xyz="0 0 0" rpy="0 0 0"/>
-        </xacro:inertial_cylinder>
+        <inertial>
+            <mass
+              value="7.5613" />
+            <inertia
+              ixx="0.063626"
+              ixy="0"
+              ixz="0"
+              iyy="0.063626"
+              iyz="0"
+              izz="0.11054" />
+          </inertial>
 	</link>
     <gazebo reference="front_right_wheel_move">
@@ -140,5 +167,9 @@
         <origin xyz="${front_rear_sep + (chasis_x - front_rear_sep)/2} ${wheel_sep/2 + wheel_thickness} 0" rpy="0 0 0" />
         <axis xyz="0 0 1"/>
-        <limit effort="100" velocity="1" lower="-${max_steer}" upper="${max_steer}"/>
+        <limit
+        lower="-0.69"
+        upper="0.69"
+        effort="0"
+        velocity="0" />
     </joint>
     <link name="front_left_wheel_rotate">
@@ -153,10 +184,17 @@
             <origin xyz="0 0 0" rpy="${-pi/2} 0 0" />
 		    <geometry>
-                <cylinder length="${wheel_thickness}" radius="${wheel_radius}"/>
-            </geometry>
-		</collision>
-		<xacro:inertial_cylinder mass="${wheel_mass}" length="${wheel_thickness}" radius="${wheel_radius}">
-            <origin xyz="0 0 0" rpy="${-pi/2} 0 0"/>
-        </xacro:inertial_cylinder>
+                <sphere radius="${wheel_radius}"/>
+            </geometry>
+		</collision>
+		<inertial>
+            <mass value="7.8526" />
+            <inertia
+              ixx="0.063827"
+              ixy="0"
+              ixz="0"
+              iyy="0.063827"
+              iyz="0"
+              izz="0.11091" />
+          </inertial>
 	</link>
     <gazebo reference="front_left_wheel_rotate">
@@ -174,4 +212,5 @@
         <origin xyz="0 0 0" rpy="-${pi/2} 0 0" />
         <axis xyz="0 0 1" rpy="0 0 0" />
+        <dynamics damping="0.0" friction="15"/>
     </joint>
 	<link name="front_left_wheel_move">
@@ -184,10 +223,18 @@
 		<collision>
 		    <geometry>
-                <cylinder length="${wheel_thickness}" radius="${wheel_radius}"/>
+                <sphere radius="${wheel_radius}"/>
 		    </geometry>
 		</collision>
-        <xacro:inertial_cylinder mass="${wheel_mass}" length="${wheel_thickness}" radius="${wheel_radius}">
-            <origin xyz="0 0 0" rpy="0 0 0"/>
-        </xacro:inertial_cylinder>
+        <inertial>
+            <mass
+              value="7.7007" />
+            <inertia
+              ixx="0.063724"
+              ixy="0"
+              ixz="0"
+              iyy="0.063724"
+              iyz="0"
+              izz="0.11072" />
+          </inertial>
 	</link>
     <gazebo reference="front_left_wheel_move">
@@ -204,4 +251,5 @@
         <child link="back_right_wheel"/>
         <origin xyz="${(chasis_x - front_rear_sep)/2} -${wheel_sep/2 + wheel_thickness} 0" rpy="${pi/2} 0 0" />
+        <dynamics damping="0.0" friction="15"/>
         <axis xyz="0 0 -1"/>
     </joint>
@@ -218,7 +266,15 @@
             </geometry>
 		</collision>
-		<xacro:inertial_cylinder mass="${wheel_mass}" length="${wheel_thickness}" radius="${wheel_radius}">
-            <origin xyz="0 0 0" rpy="0 0 0"/>
-        </xacro:inertial_cylinder>
+		<inertial>
+            <mass
+              value="7.7133" />
+            <inertia
+              ixx="0.06373"
+              ixy="0"
+              ixz="0"
+              iyy="0.06373"
+              iyz="0"
+              izz="0.11073" />
+          </inertial>
 	</link>
     <gazebo reference="back_right_wheel">
@@ -235,4 +291,5 @@
         <child link="back_left_wheel"/>
         <origin xyz="${(chasis_x - front_rear_sep)/2} ${wheel_sep/2 + wheel_thickness} 0" rpy="-${pi/2} 0 0" />
+        <dynamics damping="0.0" friction="15"/>
         <axis xyz="0 0 1"/>
     </joint>
@@ -249,7 +306,15 @@
             </geometry>
 		</collision>
-		<xacro:inertial_cylinder mass="${wheel_mass}" length="${wheel_thickness}" radius="${wheel_radius}">
-            <origin xyz="0 0 0" rpy="0 0 0"/>
-        </xacro:inertial_cylinder>
+		<inertial>
+            <mass
+              value="7.6692" />
+            <inertia
+              ixx="0.063699"
+              ixy="0"
+              ixz="0"
+              iyy="0.063699"
+              iyz="0"
+              izz="0.11067" />
+          </inertial>
 	</link>
     <gazebo reference="back_left_wheel">

File: hunter_sim_pkg/description/simple_urdf/ros2_control.xacro (robot description, xacro)
@@ -42,6 +42,6 @@
                 <remapping>ack_cont/odometry:=odom</remapping>
                 <remapping>ack_cont/tf_odometry:=tf</remapping>
-                <remapping>ack_cont/reference:=cmd_vel_stamped</remapping>
-                <!-- <remapping>ack_cont/reference_unstamped:=cmd_vel</remapping> -->
+                <!-- <remapping>ack_cont/reference:=cmd_vel_stamped</remapping> -->
+                <remapping>ack_cont/reference_unstamped:=cmd_vel</remapping>
             </ros>
             <parameters>$(find hunter_sim_pkg)/config/my_controllers.yaml</parameters>
