Commit message: arreglado yaml file de nav2

File: hunter_sim_pkg/description/hunter_urdf/hunter_core.xacro (robot description, xacro)
@@ -7,5 +7,5 @@
             <origin xyz="0 0 0" rpy="0 0 0"/>
             <geometry>
-                <mesh filename="file://hunter_sim_pkg/mesh/base_link.dae"/>
+                <mesh filename="file://$(find hunter_sim_pkg)/mesh/base_link.stl"/>
             </geometry>
             <material name="grey_1"/>
@@ -14,5 +14,5 @@
             <origin xyz="0 0 0" rpy="0 0 0" />
             <geometry>
-                <mesh filename="file://hunter_sim_pkg/mesh/base_link.dae" />
+                <mesh filename="file://$(hunter_sim_pkg)/mesh/base_link.stl" />
             </geometry>
         </collision>
