Commit message: added interfaz to ws

File: hunter_sim_pkg/description/simple_urdf/gps.xacro (robot description, xacro)
@@ -2,7 +2,7 @@
 <robot xmlns:xacro="http://www.ros.org/wiki/xacro"  name="robot">
     <joint name="gps_joint" type="fixed">
-        <parent link="chasis"/>
+        <parent link="base_link"/>
         <child link="gps_frame"/>
-        <origin xyz="0 0 0.6" rpy="0 0 0"/>
+        <origin xyz="-0.49 0 0.4" rpy="0 0 0"/>
     </joint>
     <link name="gps_frame">

File: hunter_sim_pkg/description/simple_urdf/imu.xacro (robot description, xacro)
@@ -12,12 +12,9 @@
           </geometry>
         </collision>
-        <xacro:inertial_cylinder mass="0.1" length="0.04" radius="0.05">
-            <origin xyz="0 0 0" rpy="0 0 0"/>
-        </xacro:inertial_cylinder>
       </link>
       <joint name="imu_joint" type="fixed">
-        <parent link="chasis"/>
+        <parent link="base_link"/>
         <child link="imu_link"/>
-        <origin xyz="0 0 0.01"/>
+        <origin xyz="0.13 0 0.61"/>
       </joint>
       <gazebo reference="imu_link">
@@ -27,5 +24,5 @@
               <remapping>~/out:=imu</remapping>
             </ros>
-            <initial_orientation_as_reference>false</initial_orientation_as_reference>
+            <initial_orientation_as_reference>true</initial_orientation_as_reference>
           </plugin>
           <always_on>true</always_on>
@@ -33,30 +30,4 @@
           <visualize>true</visualize>
          <imu>
-            <!-- <orientation>
-              <x>
-                <noise type="gaussian">
-                 <mean>0.0</mean>
-                 <stddev>-1</stddev>
-                 <bias_mean>0.0</bias_mean>
-                 <bias_stddev>-1</bias_stddev>
-               </noise>
-             </x>
-             <y>
-              <noise type="gaussian">
-               <mean>0.0</mean>
-               <stddev>-1</stddev>
-               <bias_mean>0.0</bias_mean>
-               <bias_stddev>-1</bias_stddev>
-             </noise>
-            </y>
-           <z>
-            <noise type="gaussian">
-             <mean>0.0</mean>
-             <stddev>-1</stddev>
-             <bias_mean>0.0</bias_mean>
-             <bias_stddev>-1</bias_stddev>
-           </noise>
-          </z>
-            </orientation> -->
              <angular_velocity>
                <x>

File: hunter_sim_pkg/description/simple_urdf/lidar.xacro (robot description, xacro)
@@ -2,7 +2,7 @@
 <robot xmlns:xacro="http://www.ros.org/wiki/xacro"  name="robot">
     <joint name="lidar_joint" type="fixed">
-        <parent link="chasis"/>
+        <parent link="base_link"/>
         <child link="laser_frame"/>
-        <origin xyz="0.5 0 0.6" rpy="0 0 0"/>
+        <origin xyz="0.13 0 0.61" rpy="0 0 0"/>
     </joint>
     <link name="laser_frame">

File: hunter_sim_pkg/description/simple_urdf/robot.urdf.xacro (robot description, xacro)
@@ -7,9 +7,9 @@
     <xacro:include filename="gps.xacro"/>
     <xacro:include filename="imu.xacro"/>
-    <xacro:if value="$(arg use_ros2_control)">
+    <!-- <xacro:if value="$(arg use_ros2_control)">
         <xacro:include filename="ros2_control.xacro" />
     </xacro:if>
     <xacro:unless value="$(arg use_ros2_control)">
         <xacro:include filename="gazebo_control.xacro" />
-    </xacro:unless>
+    </xacro:unless> -->
 </robot>

File: hunter_sim_pkg/description/simple_urdf/robot_core.xacro (robot description, xacro)
@@ -32,37 +32,28 @@
     <xacro:property name="mu2" value="2"/>
 	<!-- Base link -->
-    <link name="base_link">
+    <link name="base_footprint">
     </link>
 	<!-- Chasis-->
-	<joint name="chasis_joint" type="fixed">
-        <parent link="base_link"/>
-        <child link="chasis"/>
+	<joint name="base_link_joint" type="fixed">
+        <parent link="base_footprint"/>
+        <child link="base_link"/>
+        <origin xyz="0 0 0.105" rpy="0 0 0"/>
     </joint>
-    <link name="chasis">
+    <link name="base_link">
         <visual>
-            <origin xyz="${chasis_x/2} 0 ${chasis_z/2}" rpy="0 0 0"/>
-            <geometry>
+            <!-- <origin xyz="0 0 ${chasis_z/2}" rpy="0 0 0"/>  -->
+            <!-- <geometry>
             <box size="${chasis_x} ${chasis_y} ${chasis_z}"/>
             </geometry>
-            <material name="white"/>
+            <material name="white"/>  -->
         </visual>
         <collision>
-        <origin xyz="${chasis_x/2} 0 ${chasis_z/2}" rpy="0 0 0"/>
+        <!-- <origin xyz="${chasis_x/2} 0 ${chasis_z/2}" rpy="0 0 0"/>
         <geometry>
                 <box size="${chasis_x} ${chasis_y} ${chasis_z}"/>
-        </geometry>
+        </geometry>  -->
         </collision>
-        <inertial>
-            <mass value="21.02945169536679" />
-            <inertia
-              ixx="0.0332370959804736"
-              ixy="-1.013150489971E-06"
-              ixz="-0.00188859201421112"
-              iyy="0.111072002332437"
-              iyz="-5.13308150598312E-07"
-              izz="0.12660862809283" />
-          </inertial>
     </link>
-    <gazebo reference="chasis">
+    <gazebo reference="base_link">
         <kp>1000000.0</kp>
         <kd>0.1</kd>
@@ -75,257 +66,3 @@
         <fdir1 value="0 1 0"/>
     </gazebo>
-    <!--FRONT RIGHT WHEEL ROTATE-->
-    <joint name="front_right_wheel_rotate_joint" type="revolute">
-        <parent link="chasis"/>
-        <child link="front_right_wheel_rotate"/>
-        <origin xyz="${front_rear_sep + (chasis_x - front_rear_sep)/2} -${wheel_sep/2 + wheel_thickness} 0" rpy="0 0 0" />
-        <axis xyz="0 0 1"/>
-        <limit
-      lower="-0.69"
-      upper="0.69"
-      effort="0"
-      velocity="0" />
-    </joint>
-    <link name="front_right_wheel_rotate">
-        <visual>
-            <origin xyz="0 0 0" rpy="${pi/2} 0 0" />
-            <geometry>
-                <cylinder length="${wheel_thickness}" radius="${wheel_radius}"/>
-            </geometry>
-            <material name="blue"/>
-        </visual>
-		<collision>
-            <origin xyz="0 0 0" rpy="${pi/2} 0 0" />
-		    <geometry>
-                <sphere  radius="${wheel_radius}"/>
-            </geometry>
-		</collision>
-		<inertial>
-            <mass
-              value="7.696" />
-            <inertia
-              ixx="0.063704"
-              ixy="0"
-              ixz="0"
-              iyy="0.063704"
-              iyz="0"
-              izz="0.11068" />
-          </inertial>
-	</link>
-    <gazebo reference="front_right_wheel_rotate">
-        <mu1 value="${mu1}"/>
-        <mu2 value="${mu2}"/>
-        <kp  value="10000000.0" />
-        <kd  value="1.0" />
-        <fdir1 value="0 1 0"/>
-        <material>Gazebo/Blue</material>
-      </gazebo>
-    <!--FRONT RIGHT WHEEL MOVE-->
-    <joint name="front_right_wheel_move_joint" type="continuous">
-        <parent link="front_right_wheel_rotate"/>
-        <child link="front_right_wheel_move"/>
-        <origin xyz="0 0 0" rpy="${pi/2} 0 0" />
-        <axis xyz="0 0 -1" rpy="0 0 0" />
-        <dynamics damping="0.0" friction="15"/>
-    </joint>
-	<link name="front_right_wheel_move">
-        <visual>
-            <geometry>
-                <cylinder length="${wheel_thickness}" radius="${wheel_radius}"/>
-            </geometry>
-            <material name="blue"/>
-        </visual>
-		<collision>
-		    <geometry>
-                <sphere radius="${wheel_radius}"/>
-		    </geometry>
-		</collision>
-        <inertial>
-            <mass
-              value="7.5613" />
-            <inertia
-              ixx="0.063626"
-              ixy="0"
-              ixz="0"
-              iyy="0.063626"
-              iyz="0"
-              izz="0.11054" />
-          </inertial>
-	</link>
-    <gazebo reference="front_right_wheel_move">
-        <mu1 value="${mu1}"/>
-        <mu2 value="${mu2}"/>
-        <kp  value="10000000.0" />
-        <kd  value="1.0" />
-        <fdir1 value="0 1 0"/>
-        <material>Gazebo/Blue</material>
-    </gazebo>
-    <!--FRONT LEFT WHEEL ROTATE-->
-    <joint name="front_left_wheel_rotate_joint" type="revolute">
-        <parent link="chasis"/>
-        <child link="front_left_wheel_rotate"/>
-        <origin xyz="${front_rear_sep + (chasis_x - front_rear_sep)/2} ${wheel_sep/2 + wheel_thickness} 0" rpy="0 0 0" />
-        <axis xyz="0 0 1"/>
-        <limit
-        lower="-0.69"
-        upper="0.69"
-        effort="0"
-        velocity="0" />
-    </joint>
-    <link name="front_left_wheel_rotate">
-        <visual>
-            <origin xyz="0 0 0" rpy="${-pi/2} 0 0" />
-            <geometry>
-                <cylinder length="${wheel_thickness}" radius="${wheel_radius}"/>
-            </geometry>
-            <material name="blue"/>
-        </visual>
-		<collision>
-            <origin xyz="0 0 0" rpy="${-pi/2} 0 0" />
-		    <geometry>
-                <sphere radius="${wheel_radius}"/>
-            </geometry>
-		</collision>
-		<inertial>
-            <mass value="7.8526" />
-            <inertia
-              ixx="0.063827"
-              ixy="0"
-              ixz="0"
-              iyy="0.063827"
-              iyz="0"
-              izz="0.11091" />
-          </inertial>
-	</link>
-    <gazebo reference="front_left_wheel_rotate">
-        <mu1 value="${mu1}"/>
-        <mu2 value="${mu2}"/>
-        <kp  value="10000000.0" />
-        <kd  value="1.0" />
-        <fdir1 value="0 1 0"/>
-        <material>Gazebo/Blue</material>
-      </gazebo>
-    <!--LEFT RIGHT WHEEL MOVE-->
-    <joint name="front_left_wheel_move_joint" type="continuous">
-        <parent link="front_left_wheel_rotate"/>
-        <child link="front_left_wheel_move"/>
-        <origin xyz="0 0 0" rpy="-${pi/2} 0 0" />
-        <axis xyz="0 0 1" rpy="0 0 0" />
-        <dynamics damping="0.0" friction="15"/>
-    </joint>
-	<link name="front_left_wheel_move">
-        <visual>
-            <geometry>
-                <cylinder length="${wheel_thickness}" radius="${wheel_radius}"/>
-            </geometry>
-            <material name="blue"/>
-        </visual>
-		<collision>
-		    <geometry>
-                <sphere radius="${wheel_radius}"/>
-		    </geometry>
-		</collision>
-        <inertial>
-            <mass
-              value="7.7007" />
-            <inertia
-              ixx="0.063724"
-              ixy="0"
-              ixz="0"
-              iyy="0.063724"
-              iyz="0"
-              izz="0.11072" />
-          </inertial>
-	</link>
-    <gazebo reference="front_left_wheel_move">
-        <mu1 value="${mu1}"/>
-        <mu2 value="${mu2}"/>
-        <kp  value="10000000.0" />
-        <kd  value="1.0" />
-        <fdir1 value="0 1 0"/>
-        <material>Gazebo/White</material>
-      </gazebo>
-    <!--BACK RIGHT WHEEL-->
-    <joint name="back_right_wheel_joint" type="continuous">
-        <parent link="chasis"/>
-        <child link="back_right_wheel"/>
-        <origin xyz="${(chasis_x - front_rear_sep)/2} -${wheel_sep/2 + wheel_thickness} 0" rpy="${pi/2} 0 0" />
-        <dynamics damping="0.0" friction="15"/>
-        <axis xyz="0 0 -1"/>
-    </joint>
-    <link name="back_right_wheel">
-        <visual>
-            <geometry>
-                <cylinder length="${wheel_thickness}" radius="${wheel_radius}"/>
-            </geometry>
-            <material name="blue"/>
-        </visual>
-		<collision>
-		    <geometry>
-                <sphere radius="${wheel_radius}"/>
-            </geometry>
-		</collision>
-		<inertial>
-            <mass
-              value="7.7133" />
-            <inertia
-              ixx="0.06373"
-              ixy="0"
-              ixz="0"
-              iyy="0.06373"
-              iyz="0"
-              izz="0.11073" />
-          </inertial>
-	</link>
-    <gazebo reference="back_right_wheel">
-        <mu1 value="${mu1}"/>
-        <mu2 value="${mu2}"/>
-        <kp  value="10000000.0" />
-        <kd  value="1.0" />
-        <fdir1 value="0 1 0"/>
-        <material>Gazebo/Blue</material>
-      </gazebo>
-    <!--BACK LEFT WHEEL-->
-    <joint name="back_left_wheel_joint" type="continuous">
-        <parent link="chasis"/>
-        <child link="back_left_wheel"/>
-        <origin xyz="${(chasis_x - front_rear_sep)/2} ${wheel_sep/2 + wheel_thickness} 0" rpy="-${pi/2} 0 0" />
-        <dynamics damping="0.0" friction="15"/>
-        <axis xyz="0 0 1"/>
-    </joint>
-    <link name="back_left_wheel">
-        <visual>
-            <geometry>
-                <cylinder length="${wheel_thickness}" radius="${wheel_radius}"/>
-            </geometry>
-            <material name="blue"/>
-        </visual>
-		<collision>
-		    <geometry>
-                <sphere radius="${wheel_radius}"/>
-            </geometry>
-		</collision>
-		<inertial>
-            <mass
-              value="7.6692" />
-            <inertia
-              ixx="0.063699"
-              ixy="0"
-              ixz="0"
-              iyy="0.063699"
-              iyz="0"
-              izz="0.11067" />
-          </inertial>
-	</link>
-    <gazebo reference="back_left_wheel">
-        <material>Gazebo/Blue</material>
-    </gazebo>
-    <gazebo reference="left_wheel_rear">
-        <mu1 value="${mu1}"/>
-        <mu2 value="${mu2}"/>
-        <kp  value="10000000.0" />
-        <kd  value="1.0" />
-        <fdir1 value="0 1 0"/>
-        <material>Gazebo/Blue</material>
-    </gazebo>
 	</robot>
